File: kicad/gs/gs/gs.kicad_sch (KiCad schematic)
At the start: 54 parts, among them J1 Jack_12V, J2 JST_MotorAz, J3 JST_MotorEl, J4 Conn_02x10_Odd_Even, J5 PowerBreakout, J6 JST_ZeroAZ, U1 ESP32-WROOM-32-DEV, U2 MPU-9250-DEV, U3 Ai-Thinker-Ra-02, U4 L7805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

Commit message: Finished report
Other:
- company: (none) -> Author: Gary Allen
- title: (none) -> PQ Ground Station
Changed lines of the file:
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@@
 (kicad_sch (version 20230121) (generator eeschema)
   (paper "A3")
+  (title_block
+    (title "PQ Ground Station")
+    (date "2023-08-13")
+    (rev "v01")
+    (company "Author: Gary Allen")
+  )
   (junction (at 327.66 114.3) (diameter 0) (color 0 0 0 0)
   )
