File: kicad/gs_old/gs/gs.kicad_sch (KiCad schematic)
At the start: 54 parts, among them J1 Jack_12V, J2 JST_MotorAz, J3 JST_MotorEl, J4 Conn_02x10_Odd_Even, J5 PowerBreakout, J6 JST_ZeroAZ, U1 ESP32-WROOM-32-DEV, U2 MPU-9250-DEV, U3 Ai-Thinker-Ra-02, U4 L7805, U5 LD1117S33TR_SOT223, U6 L6219DS, U8 L6219DS, U9 ATGM332D-5N31-PCB

Commit message: 2nd design of GS PCB
Parts:
- removed R15: 10k, Resistor_THT:R_Axial_DIN0207_L6.3mm_D2.5mm_P10.16mm_Horizontal, symbol Device:R
- renumbered C17 to C14, C18 to C15, C14 to C16, C15 to C17, C19 to C18, C20 to C19, C16 to C20, R13 to R12, R12 to R13
Connections:
- net +24V: now also J5.3 (Pin_3)
- net +5V: now also C4.1, U1.1 (EN), U5.3 (VI)
- net 5V_Int: no longer C4.1, U5.3 (VI)
- net GND: no longer J5.3 (Pin_3)
- net M1_1A: now also J2.1 (Pin_1); no longer J2.2 (Pin_2)
- net M1_1B: now also J2.2 (Pin_2); no longer J2.1 (Pin_1)
- net M1_2A: now also J2.3 (Pin_3); no longer J2.4 (Pin_4)
- net M1_2B: now also J2.4 (Pin_4); no longer J2.3 (Pin_3)
- net M1_I01: now also U1.18 (TXD0/IO1); no longer U1.4 (IO34)
- net M1_I02: now also U1.19 (RXD0/IO3); no longer U1.9 (IO26)
- net M1_I12: now also U1.6 (IO32); no longer U1.8 (IO25)
- net M1_P1: now also U1.4 (IO34); no longer U1.6 (IO32)
- net M2_1A: now also J3.1 (Pin_1); no longer J3.2 (Pin_2)
- net M2_1B: now also J3.2 (Pin_2); no longer J3.1 (Pin_1)
- net M2_2A: now also J3.3 (Pin_3); no longer J3.4 (Pin_4)
- net M2_2B: now also J3.4 (Pin_4); no longer J3.3 (Pin_3)
- net M2_I01: now also U1.8 (IO25); no longer U1.18 (TXD0/IO1)
- net M2_I02: now also U1.9 (IO26); no longer U1.27 (IO2)
- net M2_I11: now also U1.11 (IO14); no longer U1.19 (RXD0/IO3)
- net M2_I12: now also U1.13 (IO13); no longer U1.26 (IO4)
- net M2_P1: now also U1.10 (IO27); no longer U1.20 (IO21)
- net M2_P2: now also U1.12 (IO12); no longer U1.23 (IO5)
- net RF_DIO1: now also J4.14 (Pin_14); no longer J4.1 (Pin_1)
- net RF_DIO2: now also J4.12 (Pin_12); no longer J4.5 (Pin_5)
- net RF_DIO3: now also J4.10 (Pin_10); no longer J4.3 (Pin_3)
- net RF_DIO4: now also J4.15 (Pin_15); no longer J4.16 (Pin_16)
- net RF_DIO5: now also J4.13 (Pin_13); no longer J4.14 (Pin_14)
- net RF_NRESET: now also J4.16 (Pin_16); no longer J4.7 (Pin_7)
- net RF_NSS: now also U1.20 (IO21); no longer U1.10 (IO27)
- net SPI_MISO: now also J4.11 (Pin_11); no longer J4.10 (Pin_10)
- net SPI_MOSI: now also J4.9 (Pin_9); no longer J4.8 (Pin_8)
- net SPI_SCK: now also J4.7 (Pin_7); no longer J4.12 (Pin_12)
- net BRK_GPIO12: no longer names the net of J4.4 (Pin_4)
- net BRK_GPIO12: no longer U1.12 (IO12)
- net BRK_GPIO13: no longer names the net of J4.6 (Pin_6)
- net BRK_GPIO13: no longer U1.13 (IO13)
- net BRK_GPIO14: no longer names the net of J4.2 (Pin_2)
- net BRK_GPIO14: no longer U1.11 (IO14)
- net M1_Sense1_In: no longer names the net of R5.1, R6.1, U6.23 (SENSE1)
- net M1_Sense2_In: no longer names the net of R7.1, R8.1, U6.3 (SENSE2)
- net M2_Sense1_In: no longer names the net of R11.1, R13.1, U8.23 (SENSE1)
- net M2_Sense2_In: no longer names the net of R12.1, R14.1, U8.3 (SENSE2)
- new net BRK_GPIO2: J4.1 (Pin_1), U1.27 (IO2)
- new net BRK_GPIO4: J4.3 (Pin_3), U1.26 (IO4)
- new net BRK_GPIO5: J4.5 (Pin_5), U1.23 (IO5)
- no-connect marks 11 -> 14
