File: kicad/gs_old/gs/gs.kicad_pcb (KiCad board)
At the start: 2 copper layers, 198 x 198 mm, 53 parts, among them J1 Jack_12V, J2 JST_MotorAz, J3 JST_MotorEl, J4 Conn_02x10_Odd_Even, J5 PowerBreakout, J6 JST_ZeroAZ, U1 ESP32-WROOM-32-DEV, U2 MPU-9250-DEV, U3 Ai-Thinker-Ra-02, U4 L7805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

Commit message: Exported GS Rev 4 Gerbers
Routing:
- net M2_I01: vias 2 -> 3
- net GND: vias 89 -> 178
